File: ra8875_40pin_REV-D.brd (EAGLE design)
At the start: 48.3 x 40.6 mm, 54 parts, among them J1 40PINFPCM4-1734839-0, U1 RA8875, U3 FAN5333BSX, U4 MIC5225-3.3v, U5 74HC4050, Y1 20MHz

Commit message: Updated to the latest board and schematic
Connections:
- net !INT renamed INT
- net !WAIT renamed WAIT
- net SPI_CLK renamed SCK
- net SPI_CS renamed CS
Changed lines of the file:
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@@
 <?xml version="1.0" encoding="utf-8"?>
 <!DOCTYPE eagle SYSTEM "eagle.dtd">
-<eagle version="6.3">
+<eagle version="6.4">
 <drawing>
 <settings>
@@
 <layer number="19" name="Unrouted" color="6" fill="1" visible="yes" active="yes"/>
 <layer number="20" name="Dimension" color="15" fill="1" visible="yes" active="yes"/>
-<layer number="21" name="tPlace" color="14" fill="1" visible="no" active="yes"/>
-<layer number="22" name="bPlace" color="13" fill="1" visible="no" active="yes"/>
+<layer number="21" name="tPlace" color="14" fill="1" visible="yes" active="yes"/>
+<layer number="22" name="bPlace" color="13" fill="1" visible="yes" active="yes"/>
 <layer number="23" name="tOrigins" color="15" fill="1" visible="yes" active="yes"/>
-<layer number="24" name="bOrigins" color="15" fill="1" visible="no" active="yes"/>
+<layer number="24" name="bOrigins" color="15" fill="1" visible="yes" active="yes"/>
 <layer number="25" name="tNames" color="7" fill="1" visible="no" active="yes"/>
 <layer number="26" name="bNames" color="7" fill="1" visible="no" active="yes"/>
-<layer number="27" name="tValues" color="7" fill="1" visible="yes" active="yes"/>
+<layer number="27" name="tValues" color="7" fill="1" visible="no" active="yes"/>
 <layer number="28" name="bValues" color="7" fill="1" visible="no" active="yes"/>
-<layer number="29" name="tStop" color="7" fill="3" visible="yes" active="yes"/>
+<layer number="29" name="tStop" color="7" fill="3" visible="no" active="yes"/>
 <layer number="30" name="bStop" color="7" fill="6" visible="no" active="yes"/>
 <layer number="31" name="tCream" color="7" fill="4" visible="no" active="yes"/>
@@
 <wire x1="2.278" y1="10.541" x2="2.278" y2="10.414" width="0.4064" layer="1"/>
 </signal>
-<signal name="!INT">
+<signal name="INT">
 <contactref element="U1" pad="8"/>
 <wire x1="23.146" y1="9.268" x2="23.146" y2="6.39" width="0.254" layer="1"/>
@@
 <contactref element="JP1" pad="5"/>
 </signal>
-<signal name="!WAIT">
+<signal name="WAIT">
 <contactref element="U1" pad="7"/>
 <wire x1="22.646" y1="9.268" x2="22.646" y2="6.048" width="0.254" layer="1"/>
@@
 <wire x1="28.694" y1="6.35" x2="29.837" y2="7.493" width="0.254" layer="1"/>
 </signal>
-<signal name="SPI_CLK">
+<signal name="SCK">
 <contactref element="U5" pad="3"/>
 <wire x1="30.353" y1="8.509" x2="36.314" y2="8.509" width="0.254" layer="16"/>
@@
 <wire x1="21.59" y1="3.175" x2="21.59" y2="1.905" width="0.254" layer="16"/>
 </signal>
-<signal name="SPI_CS">
+<signal name="CS">
 <contactref element="U5" pad="7"/>
 <wire x1="37.076" y1="6.985" x2="42.791" y2="12.7" width="0.254" layer="16"/>
