File: ra8875_40pin_REV-D.sch (EAGLE design)
At the start: 52 parts, among them J1 40PINFPCM4-1734839-0, U1 RA8875, U3 FAN5333BSX, U4 MIC5225-3.3v, U5 74HC4050, Y1 20MHz

Commit message: Updated to the latest board and schematic
Connections:
- net !INT renamed INT
- net !WAIT renamed WAIT
- net SPI_CLK renamed SCK
- net SPI_CS renamed CS
Other:
- moved on the sheet: C1, C10, C11, C12, C16, C17, C18, C19, C2, C20, C21, C22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
