File: Adafruit RA8875 TFT Breakout.brd (EAGLE design)
At the start: 48.3 x 40.6 mm, 54 parts, among them J1 40PINFPCM4-1734839-0, U1 RA8875, U3 FAN5333BSX, U4 MIC5225-3.3v, U5 74HC4050, Y1 20MHz

Commit message: Update board files to latest rev
Parts:
- removed D1: MM3Z24VT1G, microbuilder:SMADIODE
- added IC2: 74AHC1G125DBV, 74xx-little-us:SOT23-5
- added PLABEL0: (no value), pinguin:PLABEL0
- added PLABEL1: (no value), pinguin:PLABEL1
- added PLABEL10: (no value), pinguin:PLABEL10
- added PLABEL11: (no value), pinguin:PLABEL11
- added PLABEL12: (no value), pinguin:PLABEL12
- added PLABEL13: (no value), pinguin:PLABEL13
- added PLABEL14: (no value), pinguin:PLABEL14
- added PLABEL15: (no value), pinguin:PLABEL15
- added PLABEL16: (no value), pinguin:PLABEL16
- added PLABEL17: (no value), pinguin:PLABEL17
- added PLABEL18: (no value), pinguin:PLABEL18
- added PLABEL19: (no value), pinguin:PLABEL19
- added PLABEL2: (no value), pinguin:PLABEL2
- added PLABEL20: (no value), pinguin:PLABEL20
- added PLABEL21: (no value), pinguin:PLABEL21
- added PLABEL22: (no value), pinguin:PLABEL22
- added PLABEL23: (no value), pinguin:PLABEL23
- added PLABEL3: (no value), pinguin:PLABEL3
- added PLABEL4: (no value), pinguin:PLABEL4
- added PLABEL5: (no value), pinguin:PLABEL5
- added PLABEL6: (no value), pinguin:PLABEL6
- added PLABEL7: (no value), pinguin:PLABEL7
- added PLABEL8: (no value), pinguin:PLABEL8
- added PLABEL9: (no value), pinguin:PLABEL9
- added U$30: (no value), microbuilder:PCBFEAT-REV-040
- C1, C10, C11, C12, C5, C6, C7, C8, C9, R12, R3: device microbuilder:0805-NO -> microbuilder:0603-NO
- C16, C17, C20, C22, FB2: device microbuilder:_0805MP -> microbuilder:0805-NO
- C18, R11: device microbuilder:_0805MP -> microbuilder:0603-NO
- C19, C21: value 10µF -> 10uF; device microbuilder:_0805MP -> microbuilder:0805-NO
- C2, C3: value 20pF -> 15pF; device microbuilder:0805-NO -> microbuilder:0603-NO
- C4: value 0.1uF -> 1uF
- D3, D4: device adafruit:SOD-323F -> microbuilder:SOD-323_MINI
- FID1, FID2, FID3: value FIDUCIAL"" -> FIDUCIAL_1MM
- J1: value 40PINFPCM4-1734839-0 -> 40PINFPC_GENERIC; device adafruit:4-1734839-0 -> adafruit_display:FPC_40
- R1: value 3Ω -> 2Ω; device microbuilder:_0805MP -> microbuilder:0805-NO
- R10, R9: value 12Ω -> 8.2Ω; device microbuilder:_0805MP -> microbuilder:0805-NO
- U$21, U$22, U$23, U$24: device microbuilder:MOUNTINGHOLE_2.5_PLATED -> adafruit_electromech:MOUNTINGHOLE_2.5_PLATED
- U3: value FAN5333BSX -> TPS61169; device microbuilder:SOT23-5@1 -> adafruit_power:SC70-5
- U4: value MIC5225-3.3v -> AP2127K-3.3; device microbuilder:SOT23-5 -> adafruit_power:SOT23-5
- U5: device microbuilder:SOIC16 -> microbuilder:TSSOP16
- moved R1 9.44 mm to (10.7, 29.1)
- moved SJ2 6.13 mm to (8.76, 29.0), flipped to the top, turned to 90 degrees
- moved R9 5.08 mm to (6.73, 29.0), turned to 90 degrees
- moved R10 4.84 mm to (2.67, 29.0), turned to 90 degrees
- moved C18 4.33 mm to (2.41, 26.3)
- moved SJ1 4.26 mm to (4.70, 29.0), flipped to the top, turned to 90 degrees
- moved D3 3.50 mm to (3.30, 17.5), turned to 90 degrees
- moved U3 2.71 mm to (2.28, 23.7)
- moved D4 2.62 mm to (1.52, 17.5), turned to 90 degrees
- moved R11 2.57 mm to (2.40, 20.6)
- moved J1 1.52 mm to (28.4, 36.1)
- moved C21 1.40 mm to (14.2, 33.1)
- moved C16 1.30 mm to (7.87, 17.8)
- moved C22 1.14 mm to (8.63, 10.7)
- moved C1 0.99 mm to (15.2, 28.1), turned to 90 degrees
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Connections:
- new net RA_MISO: IC2.2, U1.42
- net +24V: no longer D1.C
- net +3V3: now also IC2.5
- net GND: now also IC2.3
- net LEDK: no longer D1.A
- net MISO: now also IC2.4; no longer U1.42
- net SPI_CS_3V: now also IC2.1
Routing:
- net GND: track 147.5 -> 91.3 mm, vias 25 -> 28
- net RA_MISO: track 0.00 -> 12.2 mm, vias 0 -> 2
- net MISO: track 40.1 -> 29.0 mm
- net N$24: track 10.1 -> 3.00 mm, vias 1 -> 0
- net SCK: track 45.8 -> 39.1 mm
- net +24V: track 19.0 -> 15.3 mm
- net PWM0: track 32.3 -> 35.5 mm
- net SPI_CS_3V: track 7.37 -> 10.2 mm
- net R5: track 9.22 -> 6.55 mm
- net RESET: track 27.7 -> 30.0 mm
- net MOSI: track 35.5 -> 33.9 mm
- net VIN: track 35.6 -> 37.2 mm
- net SPI_CLK_3V: track 8.82 -> 7.27 mm
- net N$3: track 9.45 -> 8.09 mm
- net BACKLITE: track 18.8 -> 20.2 mm
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- added copper zone on layer 1, net GND
Other:
- board text added: "+100"
- board text added: "+25"
- board text removed: "+100mA"
- board text removed: "+25mA"
