File: Adafruit RA8875 TFT Breakout.sch (EAGLE design)
At the start: 52 parts, among them J1 40PINFPCM4-1734839-0, U1 RA8875, U3 FAN5333BSX, U4 MIC5225-3.3v, U5 74HC4050, Y1 20MHz

Commit message: Update board files to latest rev
Parts:
- removed D1: MM3Z24VT1G, microbuilder:DIODESMA
- added IC2: 74AHC1G125DBV, 74xx-little-us:74AHC1G125DBV
- C1, C10, C11, C12, C5, C6, C7, C8, C9: device microbuilder:CAP_CERAMIC0805-NOOUTLINE -> microbuilder:CAP_CERAMIC0603_NO
- C16, C17, C20, C22: device microbuilder:CAP_CERAMIC_0805MP -> microbuilder:CAP_CERAMIC0805-NOOUTLINE
- C18: device microbuilder:CAP_CERAMIC_0805MP -> microbuilder:CAP_CERAMIC0603_NO
- C19, C21: value 10µF -> 10uF; device microbuilder:CAP_CERAMIC_0805MP -> microbuilder:CAP_CERAMIC0805-NOOUTLINE
- C2, C3: value 20pF -> 15pF; device microbuilder:CAP_CERAMIC0805-NOOUTLINE -> microbuilder:CAP_CERAMIC0603_NO
- C4: value 0.1uF -> 1uF
- D3, D4: device adafruit:DIODESOD-323F -> microbuilder:DIODE_SOD323MINI
- FB2: device microbuilder:FERRITE_0805MP -> microbuilder:FERRITE-0805NO
- FID1, FID2, FID3: value FIDUCIAL"" -> FIDUCIAL_1MM; device microbuilder:FIDUCIAL"" -> microbuilder:FIDUCIAL_1MM
- J1: value 40PINFPCM4-1734839-0 -> 40PINFPC_GENERIC; device adafruit:40PINFPCM4-1734839-0 -> adafruit_display:40PINFPC_GENERIC
- R1: value 3Ω -> 2Ω; device microbuilder:RESISTOR_0805MP -> microbuilder:RESISTOR0805_NOOUTLINE
- R10, R9: value 12Ω -> 8.2Ω; device microbuilder:RESISTOR_0805MP -> microbuilder:RESISTOR0805_NOOUTLINE
- R11: device microbuilder:RESISTOR_0805MP -> microbuilder:RESISTOR_0603_NOOUT
- R12, R3: device microbuilder:RESISTOR0805_NOOUTLINE -> microbuilder:RESISTOR_0603_NOOUT
- U$21, U$22, U$23, U$24: device microbuilder:MOUNTINGHOLE2.5 -> adafruit_electromech:MOUNTINGHOLE2.5
- U3: value FAN5333BSX -> TPS61169; device microbuilder:FAN5331 -> adafruit_power:VREG_BOOST_5PIN_SC70
- U4: value MIC5225-3.3v -> AP2127K-3.3; device microbuilder:VREG_SOT23-5 -> adafruit_power:VREG_SOT23-5
- U5: device microbuilder:74HC4050D -> microbuilder:74HC4050DTSSOP
Connections:
- new net RA_MISO: IC2A.I, U1.SDO
- net +24V: no longer D1.C
- net +3V3: now also IC2P.VCC
- net GND: now also IC2P.GND
- net LEDK: no longer D1.A
- net MISO: now also IC2A.O; no longer U1.SDO
- net SPI_CS_3V: now also IC2A.OE
Other:
- moved on the sheet: C1, C10, C11, C12, C16, C17, C18, C19, C2, C20, C21, C22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
